File: Avionics-GPSBoard/Connectors.kicad_sch (KiCad schematic)
At the start: 4 parts, among them J7 QSH-030-01-L-D-A, J8 QTH-030-01-L-D-A

Commit message: Add bus protection, additional routing, schematic cleanup
Connections:
- net SPI0_CLK renamed Pin_29
- net SPI0_MISO renamed Pin_33
- net SPI0_MOSI renamed Pin_31
Changed lines of the file:
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@@
 		(comment 1 "N. Khera")
 	)
-	(text_box "Connecting mounting pins to GND here"
+	(text_box "TODO: Figure out how to handle CLK and PPS"
 		(exclude_from_sim no)
-		(at 245.11 126.365 0)
+		(at 134.62 147.32 0)
 		(size 22.86 8.89)
 		(margins 0.9525 0.9525 0.9525 0.9525)
@@
 	(wire
 		(pts
-			(xy 90.17 95.25) (xy 105.41 95.25)
-		)
-		(stroke
-			(width 0)
-			(type default)
-		)
-	)
-	(wire
-		(pts
 			(xy 135.89 80.01) (xy 135.89 77.47)
 		)
@@
 	(wire
 		(pts
-			(xy 157.48 95.25) (xy 172.72 95.25)
-		)
-		(stroke
-			(width 0)
-			(type default)
-		)
-	)
-	(wire
-		(pts
 			(xy 86.36 92.71) (xy 105.41 92.71)
 		)
@@
 	(wire
 		(pts
-			(xy 90.17 100.33) (xy 105.41 100.33)
-		)
-		(stroke
-			(width 0)
-			(type default)
-		)
-	)
-	(wire
-		(pts
 			(xy 86.36 80.01) (xy 105.41 80.01)
 		)
@@
 	(wire
 		(pts
-			(xy 90.17 97.79) (xy 105.41 97.79)
-		)
-		(stroke
-			(width 0)
-			(type default)
-		)
-	)
-	(wire
-		(pts
 			(xy 135.89 64.77) (xy 118.11 64.77)
 		)
@@
 	(wire
 		(pts
-			(xy 157.48 97.79) (xy 172.72 97.79)
-		)
-		(stroke
-			(width 0)
-			(type default)
-		)
-	)
-	(wire
-		(pts
 			(xy 153.67 82.55) (xy 153.67 80.01)
 		)
@@
 	(wire
 		(pts
-			(xy 157.48 100.33) (xy 172.72 100.33)
-		)
-		(stroke
-			(width 0)
-			(type default)
-		)
-	)
-	(wire
-		(pts
 			(xy 86.36 69.85) (xy 105.41 69.85)
 		)
@@
 			(width 0)
 			(type default)
-		)
-	)
-	(label "SPI0_MISO"
-		(at 90.17 100.33 0)
-		(effects
-			(font
-				(size 1.27 1.27)
-			)
-			(justify left bottom)
 		)
 	)
@@
 		)
 	)
+	(label "Pin_31"
+		(at 172.72 97.79 180)
+		(effects
+			(font
+				(size 1.27 1.27)
+			)
+			(justify right bottom)
+		)
+	)
 	(label "Pin_54"
 		(at 185.42 125.73 0)
@@
 		)
 	)
+	(label "Pin_31"
+		(at 105.41 97.79 180)
+		(effects
+			(font
+				(size 1.27 1.27)
+			)
+			(justify right bottom)
+		)
+	)
 	(label "Pin_42"
 		(at 118.11 110.49 0)
@@
 		)
 	)
-	(label "SPI0_MOSI"
-		(at 157.48 97.79 0)
-		(effects
-			(font
-				(size 1.27 1.27)
-			)
-			(justify left bottom)
-		)
-	)
 	(label "Pin_54"
 		(at 118.11 125.73 0)
@@
 		)
 	)
-	(label "SPI0_CLK"
-		(at 90.17 95.25 0)
-		(effects
-			(font
-				(size 1.27 1.27)
-			)
-			(justify left bottom)
-		)
-	)
 	(label "Pin_58"
 		(at 118.11 130.81 0)
@@
 		)
 	)
-	(label "SPI0_MISO"
-		(at 157.48 100.33 0)
-		(effects
-			(font
-				(size 1.27 1.27)
-			)
-			(justify left bottom)
-		)
-	)
 	(label "CLKOUT"
 		(at 90.17 113.03 0)
@@
 		)
 	)
+	(label "Pin_33"
+		(at 105.41 100.33 180)
+		(effects
+			(font
+				(size 1.27 1.27)
+			)
+			(justify right bottom)
+		)
+	)
 	(label "Pin_56"
 		(at 118.11 128.27 0)
@@
 		)
 	)
-	(label "SPI0_CLK"
-		(at 157.48 95.25 0)
-		(effects
-			(font
-				(size 1.27 1.27)
-			)
-			(justify left bottom)
+	(label "Pin_33"
+		(at 172.72 100.33 180)
+		(effects
+			(font
+				(size 1.27 1.27)
+			)
+			(justify right bottom)
 		)
 	)
@@
 		)
 	)
-	(label "SPI0_MOSI"
-		(at 90.17 97.79 0)
-		(effects
-			(font
-				(size 1.27 1.27)
-			)
-			(justify left bottom)
-		)
-	)
 	(label "Pin_48"
 		(at 118.11 118.11 0)
@@
 		)
 	)
+	(label "Pin_29"
+		(at 172.72 95.25 180)
+		(effects
+			(font
+				(size 1.27 1.27)
+			)
+			(justify right bottom)
+		)
+	)
+	(label "Pin_29"
+		(at 105.41 95.25 180)
+		(effects
+			(font
+				(size 1.27 1.27)
+			)
+			(justify right bottom)
+		)
+	)
