File: Avionics-GPSBoard/Avionics-GPSBoard.kicad_sch (KiCad schematic)
At the start: 4 parts

Commit message: Status LEDs, resistor calcs
Other:
- sheet MCU_IO ports: added RF_REG_EN; removed RF_REG_SHDN
- sheet RF Receiver ports: added REG_EN; removed REG_nSHDN
Changed lines of the file:
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@@
 		(comment 1 "N. Khera")
+	)
+	(text_box "TODO: Verify"
+		(exclude_from_sim no)
+		(at 12.7 135.7517 0)
+		(size 21.59 3.9483)
+		(margins 0.9525 0.9525 0.9525 0.9525)
+		(stroke
+			(width 0)
+			(type solid)
+			(color 255 0 0 1)
+		)
+		(fill
+			(type color)
+			(color 255 2 10 0.2)
+		)
+		(effects
+			(font
+				(size 1.27 1.27)
+				(color 255 0 0 1)
+			)
+			(justify left top)
+		)
+	)
+	(text_box "TODO: Verify"
+		(exclude_from_sim no)
+		(at 78.74 199.39 0)
+		(size 21.59 3.9483)
+		(margins 0.9525 0.9525 0.9525 0.9525)
+		(stroke
+			(width 0)
+			(type solid)
+			(color 255 0 0 1)
+		)
+		(fill
+			(type color)
+			(color 255 2 10 0.2)
+		)
+		(effects
+			(font
+				(size 1.27 1.27)
+				(color 255 0 0 1)
+			)
+			(justify left top)
+		)
+	)
+	(text_box "TODO: Verify"
+		(exclude_from_sim no)
+		(at 12.7 88.9 0)
+		(size 21.59 3.9483)
+		(margins 0.9525 0.9525 0.9525 0.9525)
+		(stroke
+			(width 0)
+			(type solid)
+			(color 255 0 0 1)
+		)
+		(fill
+			(type color)
+			(color 255 2 10 0.2)
+		)
+		(effects
+			(font
+				(size 1.27 1.27)
+				(color 255 0 0 1)
+			)
+			(justify left top)
+		)
+	)
+	(text_box "TODO: Verify"
+		(exclude_from_sim no)
+		(at 154.94 105.41 0)
+		(size 21.59 3.9483)
+		(margins 0.9525 0.9525 0.9525 0.9525)
+		(stroke
+			(width 0)
+			(type solid)
+			(color 255 0 0 1)
+		)
+		(fill
+			(type color)
+			(color 255 2 10 0.2)
+		)
+		(effects
+			(font
+				(size 1.27 1.27)
+				(color 255 0 0 1)
+			)
+			(justify left top)
+		)
+	)
+	(text_box "TODO: Verify"
+		(exclude_from_sim no)
+		(at 35.56 232.41 0)
+		(size 21.59 3.9483)
+		(margins 0.9525 0.9525 0.9525 0.9525)
+		(stroke
+			(width 0)
+			(type solid)
+			(color 255 0 0 1)
+		)
+		(fill
+			(type color)
+			(color 255 2 10 0.2)
+		)
+		(effects
+			(font
+				(size 1.27 1.27)
+				(color 255 0 0 1)
+			)
+			(justify left top)
+		)
+	)
+	(text_box "TODO: Verify"
+		(exclude_from_sim no)
+		(at 116.84 231.14 0)
+		(size 21.59 3.9483)
+		(margins 0.9525 0.9525 0.9525 0.9525)
+		(stroke
+			(width 0)
+			(type solid)
+			(color 255 0 0 1)
+		)
+		(fill
+			(type color)
+			(color 255 2 10 0.2)
+		)
+		(effects
+			(font
+				(size 1.27 1.27)
+				(color 255 0 0 1)
+			)
+			(justify left top)
+		)
 	)
 	(junction
@@
 	(wire
 		(pts
-			(xy 66.04 208.28) (xy 116.84 208.28)
+			(xy 66.04 213.36) (xy 116.84 213.36)
 		)
 		(stroke
@@
 	(wire
 		(pts
-			(xy 66.04 203.2) (xy 116.84 203.2)
+			(xy 66.04 207.01) (xy 116.84 207.01)
 		)
 		(stroke
@@
 	(wire
 		(pts
-			(xy 66.04 213.36) (xy 116.84 213.36)
+			(xy 66.04 215.9) (xy 116.84 215.9)
 		)
 		(stroke
@@
 		)
 		(pin "RF_nIDLE" output
-			(at 116.84 213.36 180)
-			(effects
-				(font
-					(size 1.27 1.27)
-				)
-				(justify left)
-			)
-		)
-		(pin "RF_REG_SHDN" output
-			(at 116.84 203.2 180)
+			(at 116.84 215.9 180)
 			(effects
 				(font
@@
 		)
 		(pin "RF_CFG_BUS_nEN" output
-			(at 116.84 208.28 180)
+			(at 116.84 213.36 180)
 			(effects
 				(font
@@
 		(pin "WDT_OUT" output
 			(at 116.84 128.27 180)
+			(effects
+				(font
+					(size 1.27 1.27)
+				)
+				(justify left)
+			)
+		)
+		(pin "RF_REG_EN" output
+			(at 116.84 207.01 180)
 			(effects
 				(font
@@
 		)
 		(pin "CFG_BUS_nEN" input
-			(at 66.04 208.28 0)
+			(at 66.04 213.36 0)
 			(effects
 				(font
@@
 		)
 		(pin "nIDLE" input
-			(at 66.04 213.36 0)
-			(effects
-				(font
-					(size 1.27 1.27)
-				)
-				(justify right)
-			)
-		)
-		(pin "REG_nSHDN" input
-			(at 66.04 203.2 0)
-			(effects
-				(font
+			(at 66.04 215.9 0)
+			(effects
+				(font
+					(size 1.27 1.27)
+				)
+				(justify right)
+			)
+		)
+		(pin "REG_EN" input
+			(at 66.04 207.01 0)
+			(effects
+				(font
