File: Avionics-GPSBoard/MCU_IO.kicad_sch (KiCad schematic)
At the start: 22 parts, among them J1 DF40HC(3.0)-70DS-0.4V, J2 TC2050, J3 DF40HC(3.0)-70DS-0.4V

Commit message: Add bus protection, additional routing, schematic cleanup
Parts:
- added D11, D12, D13, D14, D15, D16: LED_G_0603_LTST-C190KRKT, LED_SMD:LED_0603_1608Metric, symbol Device:LED_Small_Filled
- added R91, R92, R93, R94, R95, R96: 2.2k, Resistor_SMD:R_0603_1608Metric, symbol Device:R_Small
Connections:
- net GND: now also D11.1 (K), D12.1 (K), D13.1 (K), D14.1 (K), D15.1 (K), D16.1 (K)
- new net: D16.2 (A), R96.2
- new net: D15.2 (A), R95.2
- new net: D12.2 (A), R92.2
- new net: D13.2 (A), R93.2
- new net: D14.2 (A), R94.2
- new net: D11.2 (A), R91.2

Commit message: Status LEDs, resistor calcs
Parts:
- R91, R92, R93, R94, R95, R96: CalcVal R_{L} -> (none)
Connections:
- net DIGIO080_B: now also R93.1
- net DIGIO081_B: now also R96.1
- net DIGIO082_B: now also R92.1
- net DIGIO083_B: now also R95.1
- net DIGIO084_B: now also R91.1
- net DIGIO085_B: now also R94.1
Other:
- note added: "Bank 8: Status LEDs"
