File: Avionics-GPSBoard/PowerInput.kicad_sch (KiCad schematic)
At the start: 20 parts, among them J5 205338-0004, J6 282834-4, U7 INA226-Q1, U8 TPS259474LRPW

Commit message: Status LEDs, resistor calcs
Parts:
- C64: value 100n -> 2n2
- R36, R38: now fitted; now in the parts list
- R37, R39: now not fitted; now left out of the parts list
- R41: value 649k -> 330k
- R42: value 100k -> 51k
- R43: value 2k7 -> 1k2
Other:
- note added: "I2C Addr = 0x45"
- note removed: "I2C Addr = 0x40"
- moved on the sheet: R40
Changed lines of the file:
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@@
 		(comment 1 "O. Anavekar")
 	)
-	(text "I2C Addr = 0x40"
+	(text "I2C Addr = 0x45"
 		(exclude_from_sim no)
 		(at 102.87 160.02 0)
@@
 		)
 	)
-	(text_box "TODO: Verify the math here!"
-		(exclude_from_sim no)
-		(at 209.55 89.2353 0)
-		(size 73.66 3.9483)
-		(margins 0.9525 0.9525 0.9525 0.9525)
-		(stroke
-			(width 0)
-			(type solid)
-			(color 255 0 0 1)
-		)
-		(fill
-			(type color)
-			(color 255 2 10 0.2)
-		)
-		(effects
-			(font
-				(size 1.27 1.27)
-				(color 255 0 0 1)
-			)
-			(justify left top)
-		)
-	)
-	(text_box "Design Requirements:\n1) [System voltage] VBATT = 6.0V - 8.4V\n2) [System overvoltage] VBATT_OV = 9.0V (600mV more than lipo max)\n3) [System max current] ILIM = 2.5A\n4) [Soft start current] I_SS = 0.5A\n4) [Load transient blanking interval] t_iob = 1ms\n\nOvervoltage:\n\nVBATT_OV = 1.2V * (1 + (RA / RB)\nRA = 649K\nRB = 100K\nVBATT_OV = 8.988V\n\nSoft Start:\nI_{SS} = C_bulk * SR\nC_{bulk} ~= 80uF (20uF for 4 DCDCs)\nSR = 6.25V/ms\nC_{S} = 2000 / SR ~= 330pF\n\nSoft Start Power Dissipation:\nPD_{SS} = (I_SS * VBATT) / 2 = 2.1W\n\nCurrent Limit:\nR_{ILM} = 3334 / 2.5A ~= 1.33K\n\nOvercurrent Blanking Interval:\nC_{O} = (t_iob * 1.8uA) / 1.51V ~= 1.2nF\n\n\nFault Logic:\n- Overcurrent response = circuit breaker\n- Fault response = latch-off\n"
+	(text_box "Design Requirements:\n1) [System voltage] VBATT = 6.0V - 8.4V\n2) [System overvoltage] VBATT_OV = 9.0V (600mV more than lipo max)\n3) [System max current] ILIM = 2.75A\n4) [Soft start current] I_SS = 0.50A\n4) [Load transient blanking interval] t_iob = 2ms\n\nOvervoltage:\n\nVBATT_OV = 1.2V * (1 + (RA / RB)\nRA = 330K\nRB = 51K\nVBATT_OV = 8.965V\n\nSoft Start:\nI_{SS} = C_bulk * SR\nC_{bulk} ~= 80uF (20uF for 4 DCDCs)\nSR = 6.25V/ms\nC_{S} = 2000 / SR ~= 330pF\n\nSoft Start Power Dissipation:\nPD_{SS} = (I_SS * VBATT) / 2 = 2.1W\n\nCurrent Limit:\nR_{ILM} = 3334 / 2.75A ~= 1.2k\n\nOvercurrent Blanking Interval:\nC_{O} = (t_iob * 1.8uA) / 1.51V ~= 2.2nF\n\n\nFault Logic:\n- Overcurrent response = circuit breaker\n- Fault response = latch-off\n"
 		(exclude_from_sim no)
 		(at 209.55 94.4536 0)
@@
 		)
 	)
-	(text_box "TODO: Ensure no collisions w/ other sensors on bus!!"
-		(exclude_from_sim no)
-		(at 101.6 170.5371 0)
-		(size 22.86 8.5329)
-		(margins 0.9525 0.9525 0.9525 0.9525)
-		(stroke
-			(width 0)
-			(type solid)
-			(color 255 0 0 1)
-		)
-		(fill
-			(type color)
-			(color 255 2 10 0.2)
-		)
-		(effects
-			(font
-				(size 1.27 1.27)
-				(color 255 0 0 1)
-			)
-			(justify left top)
-		)
-	)
 	(text_box "Power monitor placed on BUS 3V3 supply to allow continuous current monitoring even when system is unpowered."
 		(exclude_from_sim no)
@@
 	(wire
 		(pts
-			(xy 157.48 81.28) (xy 172.085 81.28)
+			(xy 167.005 90.17) (xy 152.4 90.17)
 		)
 		(stroke
@@
 	(wire
 		(pts
-			(xy 157.48 81.28) (xy 157.48 83.82)
+			(xy 167.005 90.17) (xy 167.005 92.71)
 		)
 		(stroke
@@
 	(wire
 		(pts
-			(xy 157.48 90.17) (xy 157.48 88.9)
+			(xy 167.005 99.06) (xy 167.005 97.79)
 		)
 		(stroke
@@
 	)
 	(label "SYS_ENABLE"
-		(at 157.48 81.28 0)
+		(at 167.005 90.17 180)
 		(effects
 			(font
 				(size 1.27 1.27)
 			)
-			(justify left bottom)
+			(justify right bottom)
 		)
 	)
@@
 	(hierarchical_label "SYS_ENABLE"
 		(shape input)
-		(at 172.085 81.28 0)
+		(at 152.4 90.17 180)
 		(effects
 			(font
 				(size 1.27 1.27)
 			)
-			(justify left)
+			(justify right)
 		)
 	)
@@
 		(body_style 1)
 		(exclude_from_sim no)
-		(in_bom no)
+		(in_bom yes)
 		(on_board yes)
 		(in_pos_files yes)
-		(dnp yes)
+		(dnp no)
 		(property "Reference" "R36"
 			(at 83.82 158.115 0)
@@
 			)
 		)
-		(property "Value" "649k"
+		(property "Value" "330k"
 			(at 171.45 51.308 0)
 			(show_name no)
@@
 		(body_style 1)
 		(exclude_from_sim no)
-		(in_bom yes)
+		(in_bom no)
 		(on_board yes)
-		(in_pos_files yes)
-		(dnp no)
+		(in_pos_files no)
+		(dnp yes)
 		(property "Reference" "R39"
 			(at 96.52 168.275 0)
@@
 			)
 		)
-		(property "Value" "2k7"
+		(property "Value" "1k2"
 			(at 243.84 66.548 0)
 			(show_name no)
@@
 			)
 		)
-		(property "Value" "100n"
+		(property "Value" "2n2"
 			(at 254.762 66.294 0)
 			(show_name no)
@@
 	(symbol
 		(lib_id "Device:R_Small")
-		(at 157.48 86.36 180)
+		(at 167.005 95.25 0)
+		(mirror x)
 		(unit 1)
 		(body_style 1)
@@
 		(dnp no)
 		(property "Reference" "R40"
-			(at 158.75 84.836 0)
+			(at 165.735 93.726 0)
 			(show_name no)
 			(do_not_autoplace no)
@@
 		)
 		(property "Value" "10k"
-			(at 158.75 86.868 0)
+			(at 165.735 95.758 0)
 			(show_name no)
 			(do_not_autoplace no)
@@
 		)
 		(property "Footprint" "Resistor_SMD:R_0603_1608Metric"
-			(at 157.48 86.36 0)
+			(at 167.005 95.25 0)
 			(hide yes)
 			(show_name no)
@@
 		)
 		(property "Datasheet" ""
-			(at 157.48 86.36 0)
+			(at 167.005 95.25 0)
 			(hide yes)
 			(show_name no)
@@
 		)
 		(property "Description" "Resistor, small symbol"
-			(at 157.48 86.36 0)
+			(at 167.005 95.25 0)
 			(hide yes)
 			(show_name no)
@@
 		)
 		(property "MPN" "C237112"
-			(at 157.48 86.36 0)
+			(at 167.005 95.25 0)
 			(hide yes)
 			(show_name no)
@@
 		)
 		(property "Arrow Part Number" ""
-			(at 157.48 86.36 0)
+			(at 167.005 95.25 0)
 			(hide yes)
 			(show_name no)
@@
 		)
 		(property "Arrow Price/Stock" ""
-			(at 157.48 86.36 0)
+			(at 167.005 95.25 0)
 			(hide yes)
 			(show_name no)
@@
 		)
 		(property "Height" ""
-			(at 157.48 86.36 0)
+			(at 167.005 95.25 0)
 			(hide yes)
 			(show_name no)
@@
 		)
 		(property "Mouser Part Number" ""
-			(at 157.48 86.36 0)
+			(at 167.005 95.25 0)
 			(hide yes)
 			(show_name no)
@@
 		)
 		(property "Mouser Price/Stock" ""
-			(at 157.48 86.36 0)
+			(at 167.005 95.25 0)
 			(hide yes)
 			(show_name no)
@@
 		)
 		(property "STANDARD" ""
-			(at 157.48 86.36 0)
+			(at 167.005 95.25 0)
 			(hide yes)
 			(show_name no)
@@
 		)
 		(property "Sim.Device" ""
-			(at 157.48 86.36 0)
+			(at 167.005 95.25 0)
 			(hide yes)
 			(show_name no)
@@
 		)
 		(property "Sim.Type" ""
-			(at 157.48 86.36 0)
+			(at 167.005 95.25 0)
 			(hide yes)
 			(show_name no)
@@
 			)
 		)
-		(property "Value" "100k"
+		(property "Value" "51k"
 			(at 171.45 61.468 0)
 			(show_name no)
@@
 		(body_style 1)
 		(exclude_from_sim no)
-		(in_bom no)
+		(in_bom yes)
 		(on_board yes)
 		(in_pos_files yes)
-		(dnp yes)
+		(dnp no)
 		(property "Reference" "R38"
 			(at 96.52 158.115 0)
@@
 		(body_style 1)
 		(exclude_from_sim no)
-		(in_bom yes)
+		(in_bom no)
 		(on_board yes)
-		(in_pos_files yes)
-		(dnp no)
+		(in_pos_files no)
+		(dnp yes)
 		(property "Reference" "R37"
 			(at 83.82 168.275 0)
@@
 	(symbol
 		(lib_id "power:GND")
-		(at 157.48 90.17 0)
+		(at 167.005 99.06 0)
+		(mirror y)
 		(unit 1)
 		(body_style 1)
@@
 		(dnp no)
 		(property "Reference" "#PWR0102"
-			(at 157.48 96.52 0)
+			(at 167.005 105.41 0)
 			(hide yes)
 			(show_name no)
@@
 		)
 		(property "Value" "GND"
-			(at 157.48 93.98 0)
+			(at 167.005 102.87 0)
 			(show_name no)
 			(do_not_autoplace no)
@@
 		)
 		(property "Footprint" ""
-			(at 157.48 90.17 0)
+			(at 167.005 99.06 0)
 			(hide yes)
 			(show_name no)
@@
 		)
 		(property "Datasheet" ""
-			(at 157.48 90.17 0)
+			(at 167.005 99.06 0)
 			(hide yes)
 			(show_name no)
@@
 		)
 		(property "Description" "Power symbol creates a global label with name \"GND\" , ground"
-			(at 157.48 90.17 0)
+			(at 167.005 99.06 0)
 			(hide yes)
 			(show_name no)
