File: Avionics-GPSBoard/RFReceiver.kicad_sch (KiCad schematic)
At the start: 47 parts, among them U12 MAX2769BETI_V_T, U13 TPS7A20285PDBVR, U14 TPS7A20285PDBVR, U15 D32G-016_368M, U16 TXV0106-Q1, U17 TXV0106-Q1

Commit message: Add bus protection, additional routing, schematic cleanup
Parts:
- AE1: footprint Connector_Coaxial:SMA_Amphenol_132134-11_Vertical -> Connector_Coaxial:MMCX_Molex_73415-0961_Horizontal_0.8mm-PCB
Changed lines of the file:
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@@
 			)
 		)
-		(property "Footprint" "Connector_Coaxial:SMA_Amphenol_132134-11_Vertical"
+		(property "Footprint" "Connector_Coaxial:MMCX_Molex_73415-0961_Horizontal_0.8mm-PCB"
 			(at 55.88 157.48 0)
 			(hide yes)

Commit message: Additional layout/cleanup
Connections:
- net CFG_CLK: now also U17.4 (A3); no longer U17.3 (A2)
- net CFG_DATA: now also U17.3 (A2); no longer U17.2 (A1)
- net CFG_nCS: now also U17.5 (A4); no longer U17.4 (A3)
- net SCLK: now also U17.13 (B3); no longer U17.14 (B2)
- net SDATA: now also U17.14 (B2); no longer U17.15 (B1)
- net nCS: now also U17.12 (B4); no longer U17.13 (B3)
- net nIDLE: now also U17.2 (A1); no longer U17.5 (A4)
- net nIDLE_I: now also U17.15 (B1); no longer U17.12 (B4)

Commit message: Status LEDs, resistor calcs
Connections:
- net REG_nSHDN renamed REG_EN
Changed lines of the file:
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@@
-		)
-	)
-	(text_box "Added Pi filter to make any tuning changes if needed. Stuffing inductor with 0R resistor for now"
-		(exclude_from_sim no)
-		(at 29.21 144.78 0)
-		(size 38.1 10.16)
-		(margins 0.9525 0.9525 0.9525 0.9525)
-		(stroke
-			(width 0)
-			(type solid)
-		)
-		(fill
-			(type none)
-		)
-		(effects
-			(font
-				(size 1.27 1.27)
-			)
-			(justify left top)
 		)
 	)
@@
 		)
 	)
-	(label "REG_nSHDN"
+	(label "REG_EN"
 		(at 237.49 72.39 180)
 		(effects
@@
 		)
 	)
-	(label "REG_nSHDN"
+	(label "REG_EN"
 		(at 111.76 38.1 0)
 		(effects
@@
 		)
 	)
-	(label "REG_nSHDN"
+	(label "REG_EN"
 		(at 111.76 62.23 0)
 		(effects
@@
 		)
 	)
-	(hierarchical_label "REG_nSHDN"
+	(hierarchical_label "REG_EN"
 		(shape input)
 		(at 203.2 72.39 180)
